Commit message: bug chunk

File: urdf/freddy.urdf (robot description, URDF)
Before this commit: robot freddy, 57 links, 56 joints
Links:
- link kinova_left_bracelet_link: mass 0.925 -> 1.525

Commit message: updates

File: urdf/freddy.urdf (robot description, URDF)
Before this commit: robot freddy, 57 links, 56 joints
Links:
- link kinova_left_bracelet_link: mass 1.525 -> 1.425

Commit message: uc1 working

File: urdf/freddy.urdf (robot description, URDF)
Before this commit: robot freddy, 57 links, 56 joints
Links:
- link kinova_left_bracelet_link: mass 1.425 -> 0.925
